File: main/main.kicad_pcb (KiCad board)
At the start: 2 copper layers, 64.3 x 64.1 mm, 72 parts, among them J1 Conn_01x03, J10 Conn_01x02, J11 Conn_01x02, J12 Conn_01x02, J13 Conn_01x02, J14 Conn_01x02, J15 Conn_01x02, J16 Conn_01x02, J17 Conn_01x02, J18 Conn_01x02, J19 Conn_01x02, J2 Conn_01x03, J20 Conn_01x04, J21 Conn_01x04, J22 Conn_01x06, J23 Conn_01x03, J24 Conn_01x06_Pin, J3 Conn_01x03, J4 Conn_01x03, J5 Conn_01x03, J6 Conn_01x03, J7 Conn_01x03, J8 Conn_01x03, J9 Conn_01x02, SW1 SW_DIP_x01, SW2 SW_DIP_x01, U1 XT30U-F, U2 ESP32-S3-WROOM-1, U8 CH340N, U9 AMS1117-3.3, X1 32.768KHz

Commit message: 3
Parts:
- J1, J2, J3, J4, J5, J6, J7, J8: footprint Connector:FanPinHeader_1x03_P2.54mm_Vertical -> Connector_JST:JST_XH_B3B-XH-A_1x03_P2.50mm_Vertical
- moved ADC 8.83 mm to (119.0, 138.2)
- moved C1 8.83 mm to (152.7, 138.7)
- moved BOOT 8.83 mm to (126.7, 120.2)
- moved C16 8.83 mm to (144.2, 116.6)
- moved C6 8.83 mm to (123.7, 123.9)
- moved C8 8.83 mm to (161.7, 131.2)
- moved C9 8.83 mm to (158.2, 135.7)
- moved J24 8.83 mm to (133.3, 113.2)
- moved R1 8.83 mm to (155.7, 136.2)
- moved R11 8.83 mm to (142.2, 116.7)
- moved R12 8.83 mm to (140.2, 116.7)
- moved R13 8.83 mm to (138.2, 116.7)
- moved R2 8.83 mm to (146.2, 116.7)
- moved RST 8.83 mm to (158.7, 129.2)
- moved U2 8.83 mm to (139.2, 134.6)
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- renumbered U1 to +5, J23 to ADC, J22 to Angle, SW2 to BOOT, J9 to BTN_L1, J10 to BTN_L2, J11 to BTN_L3, J12 to BTN_LS, J13 to BTN_R1, J14 to BTN_R2, J15 to BTN_R3, J16 to BTN_RS, J17 to Key1, J18 to Key2, J19 to Key3, SW1 to RST
Routing:
- net GND: track 504.9 -> 0.00 mm, vias 1 -> 0
- net /RGB_CTRL_7: track 63.5 -> 0.00 mm, vias 2 -> 0
- net /RGB_CTRL_5: track 59.6 -> 0.00 mm, vias 2 -> 0
- net /RGB_CTRL_8: track 56.6 -> 0.00 mm, vias 2 -> 0
- net /RGB_CTRL_6: track 56.1 -> 0.00 mm, vias 2 -> 0
- net +3V3: track 170.9 -> 130.3 mm, vias 3 -> 4
- net /Key_3: track 48.2 -> 9.43 mm, vias 2 -> 0
- net /RGB_CTRL_1: track 37.5 -> 0.00 mm
- net /USB_D-: track 42.9 -> 69.8 mm
- net /RGB_CTRL_2: track 26.6 -> 0.00 mm
- net /USB_D+: track 42.1 -> 66.5 mm, vias 2 -> 0
- net /RGB_CTRL_3: track 24.0 -> 0.00 mm
- net +5V: track 197.3 -> 173.4 mm
- net /UART1_RX: track 51.3 -> 75.1 mm
- net /IO37: track 21.3 -> 0.00 mm, vias 1 -> 0
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Other:
- board size 64.3 x 64.1 mm -> 64.4 x 73 mm
- board text added: "5V"
- board text added: "CTRL"
- board text added: "D+"
- board text added: "D-"
- board text added: "GND"
- board text added: "OTG"
- board text added: "UART"

Commit message: V1.0
Parts:
- added G***: LOGO, logo:shangji, F.Cu at (127.9, 107.0)
Routing:
- net /RGB_CTRL_6: track 0.00 -> 67.6 mm
- net /RGB_CTRL_5: track 0.00 -> 61.8 mm, vias 0 -> 1
- net +3V3: track 130.3 -> 190.8 mm, vias 4 -> 8
- net /Key_3: track 9.43 -> 59.5 mm, vias 0 -> 2
- net /RGB_CTRL_8: track 0.00 -> 45.6 mm, vias 0 -> 1
- net /RGB_CTRL_7: track 0.00 -> 44.4 mm, vias 0 -> 1
- net /RGB_CTRL_1: track 0.00 -> 38.4 mm, vias 0 -> 2
- net /RGB_CTRL_2: track 0.00 -> 36.7 mm, vias 0 -> 1
- net /RGB_CTRL_3: track 0.00 -> 29.6 mm, vias 0 -> 1
- net /IO37: track 0.00 -> 21.9 mm
- net /IO36: track 0.00 -> 21.7 mm
- net /IO35: track 0.00 -> 20.7 mm
- net /RGB_CTRL_4: track 0.00 -> 19.4 mm, vias 0 -> 1
- net /ADC: track 0.00 -> 12.7 mm
- net /IO21: track 0.00 -> 12.1 mm
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- added copper zone on B.Cu, net GND
- added copper zone on F.Cu, net GND
Other:
- board text added: "Ver1.0"

Commit message: V1.1
Parts:
- removed +5: XT30U-F, XT:CONN-TH_XT30U-M
- removed ADC: Conn_01x03, Connector_JST:JST_SH_BM03B-SRSS-TB_1x03-1MP_P1.00mm_Vertical
- removed BTN_LS, BTN_RS, Key3: Conn_01x02, Connector_JST:JST_SH_BM02B-SRSS-TB_1x02-1MP_P1.00mm_Vertical
- removed C10, C11, C12, C13, C14, C15, C16, C17, C18: 0.1uF, Capacitor_SMD:C_0603_1608Metric_Pad1.08x0.95mm_HandSolder
- removed J1, J2, J3, J4, J5, J6, J7, J8: Conn_01x03, Connector_JST:JST_XH_B3B-XH-A_1x03_P2.50mm_Vertical
- removed J24: Conn_01x06_Pin, Connector_PinHeader_2.54mm:PinHeader_1x06_P2.54mm_Vertical
- removed R10, R11, R12, R13, R5, R6, R7, R8, R9: 4.7K, Resistor_SMD:R_0805_2012Metric
- added C19: 0.1uF, Capacitor_SMD:C_0603_1608Metric_Pad1.08x0.95mm_HandSolder, F.Cu at (115.7, 106.0)
- added C20: 0.1uF, Capacitor_SMD:C_0603_1608Metric_Pad1.08x0.95mm_HandSolder, F.Cu at (117.0, 119.8)
- added C22: 0.1uF, Capacitor_SMD:C_0603_1608Metric_Pad1.08x0.95mm_HandSolder, F.Cu at (118.2, 133.3)
- added C23: 0.1uF, Capacitor_SMD:C_0603_1608Metric_Pad1.08x0.95mm_HandSolder, F.Cu at (116.7, 137.0)
- added C24: 0.1uF, Capacitor_SMD:C_0603_1608Metric_Pad1.08x0.95mm_HandSolder, F.Cu at (164.0, 92.9)
- added C25: 0.1uF, Capacitor_SMD:C_0603_1608Metric_Pad1.08x0.95mm_HandSolder, F.Cu at (163.2, 113.2)
- added C27: 0.1uF, Capacitor_SMD:C_0603_1608Metric_Pad1.08x0.95mm_HandSolder, F.Cu at (164.1, 128.6)
- added C28: 0.1uF, Capacitor_SMD:C_0603_1608Metric_Pad1.08x0.95mm_HandSolder, F.Cu at (162.9, 139.8)
- added R18: 4.7K, Resistor_SMD:R_0805_2012Metric, F.Cu at (117.6, 109.4)
- added R19: 4.7K, Resistor_SMD:R_0805_2012Metric, F.Cu at (117.5, 114.5)
- added R20: 4.7K, Resistor_SMD:R_0805_2012Metric, F.Cu at (118.3, 131.2)
- added R21: 4.7K, Resistor_SMD:R_0805_2012Metric, F.Cu at (119.4, 139.2)
- added R22: 4.7K, Resistor_SMD:R_0805_2012Metric, F.Cu at (161.5, 98.2)
- added R23: 4.7K, Resistor_SMD:R_0805_2012Metric, F.Cu at (162.2, 110.3)
- added R24: 4.7K, Resistor_SMD:R_0805_2012Metric, F.Cu at (162.7, 136.9)
- added R25: 4.7K, Resistor_SMD:R_0805_2012Metric, F.Cu at (143.2, 113.5)
- BTN_L1, BTN_L2, BTN_L3, BTN_R1, BTN_R2, BTN_R3: value Conn_01x02 -> Conn_01x05; footprint Connector_JST:JST_SH_BM02B-SRSS-TB_1x02-1MP_P1.00mm_Vertical -> Connector_JST:JST_XH_B5B-XH-AM_1x05_P2.50mm_Vertical
- Key1, Key2: footprint Connector_JST:JST_SH_BM02B-SRSS-TB_1x02-1MP_P1.00mm_Vertical -> Connector_JST:JST_XH_B2B-XH-AM_1x02_P2.50mm_Vertical
- moved BTN_R3 51.0 mm to (168.1, 138.5), turned to 90 degrees
- moved BTN_L3 40.6 mm to (111.8, 128.5), turned to -90 degrees
- moved BTN_R2 39.0 mm to (168.1, 120.5), turned to 90 degrees
- moved R4 34.4 mm to (150.3, 77.5), turned to 90 degrees
- moved C7 32.7 mm to (148.4, 74.6), turned to -90 degrees
- moved BTN_L2 28.6 mm to (111.8, 110.5), turned to -90 degrees
- moved BTN_R1 27.0 mm to (168.1, 102.5), turned to 90 degrees
- moved Key2 23.9 mm to (152.4, 71.6)
- moved U8 18.0 mm to (112.3, 82.2), turned to 180 degrees
- moved BTN_L1 16.6 mm to (111.8, 92.5), turned to -90 degrees
- moved J22 13.3 mm to (141.7, 71.3)
- moved R14 13.1 mm to (168.2, 74.9)
- moved C5 12.1 mm to (128.5, 78.0)
- moved R17 8.83 mm to (116.4, 74.9), turned to 180 degrees
- moved R15 8.49 mm to (165.9, 74.9)
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- renumbered Angle to J22, RST to SW1, BOOT to SW2
Connections:
- BTN_L1 pad 1: /BTN_L1 -> +5V
- BTN_L1 pad 2: GND -> /RGB_CTRL_1
- BTN_L2 pad 1: /BTN_L2 -> +5V
- BTN_L2 pad 2: GND -> Net-(BTN_L1-Pin_3)
- BTN_L3 pad 1: /BTN_L3 -> +5V
- BTN_L3 pad 2: GND -> Net-(BTN_L2-Pin_3)
- BTN_R1 pad 1: /BTN_R1 -> +5V
- BTN_R1 pad 2: GND -> /RGB_CTRL_5
- BTN_R2 pad 1: /BTN_R2 -> +5V
- BTN_R2 pad 2: GND -> Net-(BTN_R1-Pin_3)
- BTN_R3 pad 1: /BTN_R3 -> +5V
- BTN_R3 pad 2: GND -> Net-(BTN_R2-Pin_3)
- C5 pad 1: /BTN_L1 -> /Key_1
- C7 pad 1: /BTN_L2 -> /Key_2
- R3 pad 2: /BTN_L1 -> /Key_1
- R4 pad 2: /BTN_L2 -> /Key_2
Routing:
- net /RGB_CTRL_6: track 67.6 -> 0.00 mm
- net +3V3: track 190.8 -> 253.8 mm, vias 8 -> 5
- net /Key_3: track 59.5 -> 0.00 mm, vias 2 -> 0
- net /RGB_CTRL_8: track 45.6 -> 0.00 mm, vias 1 -> 0
- net /RGB_CTRL_7: track 44.4 -> 0.00 mm, vias 1 -> 0
- net /RGB_CTRL_2: track 36.7 -> 0.00 mm, vias 1 -> 0
- net /BTN_R2: track 75.6 -> 42.0 mm, vias 2 -> 1
- net /UART_TX: track 68.2 -> 100.4 mm
- net /RGB_CTRL_3: track 29.6 -> 0.00 mm, vias 1 -> 0
- net /BTN_L1: track 83.1 -> 58.2 mm
- net Net-(BTN_R1-Pin_3): track 0.00 -> 23.0 mm
- net /IO37: track 21.9 -> 0.00 mm
- net /IO36: track 21.7 -> 0.00 mm
- net Net-(BTN_R2-Pin_3): track 0.00 -> 21.7 mm
- net /IO35: track 20.7 -> 0.00 mm
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Other:
- board text added: "Ver1.1"
- board text removed: "CTRL"
- board text removed: "Ver1.0"

Commit message: V1.2
Parts:
- removed C6: 0.1uF, Capacitor_SMD:C_0603_1608Metric_Pad1.08x0.95mm_HandSolder
- moved G*** 1.32 mm to (127.9, 105.7)
Connections:
- SW2 pad 2: /Boot -> unconnected-(SW2-Pad2)
Routing:
- net /Boot: track 6.95 -> 4.02 mm
- net GND: vias 32 -> 33
Other:
- board text added: "Ver1.2"
- board text removed: "Ver1.1"

Commit message: V1.21
Parts:
- J20: footprint Connector_PinHeader_2.54mm:PinHeader_1x04_P2.54mm_Vertical -> Connector_JST:JST_XH_B4B-XH-A_1x04_P2.50mm_Vertical
- moved J20 6.62 mm to (168.7, 72.7), turned to 180 degrees
- moved R15 4.50 mm to (163.2, 78.5)
- moved R14 4.50 mm to (165.5, 78.5)
- moved SW2 0.23 mm to (126.9, 120.1)
Connections:
- J20 pad 1: /+5V_Source -> GND
- J20 pad 4: GND -> /+5V_Source
- SW2 pad 2: unconnected-(SW2-Pad2) -> /Boot
Routing:
- net /USB_D-: track 57.9 -> 53.1 mm
- net /USB_D+: track 57.9 -> 53.1 mm
- net /+5V_Source: track 80.9 -> 78.3 mm
- net Net-(J20-Pin_3): track 4.17 -> 5.09 mm
- net Net-(J20-Pin_2): track 5.46 -> 4.61 mm, vias 1 -> 0
