File: main/main.kicad_sch (KiCad schematic)
At the start: 1 part, among them U1 ESP32-S3-WROOM-1

Commit message: 2
Parts:
- removed U1: ESP32-S3-WROOM-1, RF_Module:ESP32-S3-WROOM-1, symbol RF_Module:ESP32-S3-WROOM-1
- added C1: 22uF, Capacitor_SMD:C_0805_2012Metric, symbol Device:C_Polarized
- added C2, C6, C8: 0.1uF, Capacitor_SMD:C_0603_1608Metric_Pad1.08x0.95mm_HandSolder, symbol Device:C_Polarized
- added C21, C26: 10uF, Capacitor_SMD:C_0805_2012Metric_Pad1.18x1.45mm_HandSolder, symbol Device:C_Polarized
- added C3, C4: 12pF, Capacitor_SMD:C_0603_1608Metric_Pad1.08x0.95mm_HandSolder, symbol Device:C_Polarized
- added C9: 1uF, Capacitor_SMD:C_0805_2012Metric_Pad1.18x1.45mm_HandSolder, symbol Device:C_Polarized
- added D17: SMF5.0CA, Diode_SMD:D_SOD-123F, symbol PCM_Diode_TVS_AKL:SMF5.0CA
- added D18: SMF3.3CA, Diode_SMD:D_SOD-123F, symbol PCM_Diode_TVS_AKL:SMF5.0CA
- added F3: Fuse, Fuse:Fuse_1206_3216Metric, symbol Device:Fuse
- added J1, J2, J3, J4, J5, J6, J7, J8, J9: Conn_01x03, Connector:FanPinHeader_1x03_P2.54mm_Vertical, symbol Connector_Generic:Conn_01x03
- added R1: 10K, Resistor_SMD:R_1206_3216Metric_Pad1.30x1.75mm_HandSolder, symbol PCM_Elektuur:R
- added R2: 1K, Resistor_SMD:R_1206_3216Metric_Pad1.30x1.75mm_HandSolder, symbol PCM_Elektuur:R
- added SW1, SW2: SW_DIP_x01, Button_Switch_SMD:SW_SPST_EVQPE1, symbol Switch:SW_DIP_x01
- added U2: ESP32-S3-WROOM-1, RF_Module:ESP32-S3-WROOM-1, symbol RF_Module:ESP32-S3-WROOM-1
- added U8: CH340N, Package_SO:SOP-8_3.9x4.9mm_P1.27mm, symbol Interface_USB:CH340N
- added U9: AMS1117-3.3, motor_my:SOT-223-4_L6.5-W3.5-P2.30-LS7.0-BR, symbol motor_my:AMS1117-3.3_C347222
- added X1: 32.768KHz, Crystal:Crystal_DS10_D1.0mm_L4.3mm_Vertical, symbol PCM_Crystal_AKL:Crystal_Generic
Connections:
- new net: C8.1, C9.1, R1.2 (-), SW1.2, U2.3 (EN)
- new net: C3.1, U2.8 (IO15), X1.1
- new net: C26.1, F3.1, U9.2 (VOUT(TAB)), U9.4 (TAB)
- new net: C4.1, U2.9 (IO16), X1.2
- new net: R2.1 (+), U2.16 (IO46)
- new net +3V3: C1.1, C2.1, D18.2 (A), F3.2, R1.1 (+), U2.2 (3V3), U8.5 (VCC), U8.8 (V3)
- new net +5V: C21.1, D17.2 (A), J1.2 (Pin_2), J2.2 (Pin_2), J3.2 (Pin_2), J4.2 (Pin_2), J5.2 (Pin_2), J6.2 (Pin_2), J7.2 (Pin_2), J8.2 (Pin_2), U9.3 (VIN)
- new net Boot: C6.1, SW2.2, U2.27 (IO0)
- new net Buttun: U2.39 (IO1)
- new net D+: U8.1 (UD+)
- new net D-: U8.2 (UD-)
- new net GND: C1.2, C2.2, C21.2, C26.2, C3.2, C4.2, C6.2, C8.2, C9.2, D17.1 (K), D18.1 (K), J1.3 (Pin_3), J2.3 (Pin_3), J3.3 (Pin_3), J4.3 (Pin_3), J5.3 (Pin_3), J6.3 (Pin_3), J7.3 (Pin_3), J8.3 (Pin_3), R2.2 (-), SW1.1, SW2.1, U2.1 (GND), U2.40 (GND), U2.41 (GND), U8.3 (GND), U9.1 (ADJ(GND))
- new net RGB_CTRL_1: J1.1 (Pin_1), U2.25 (IO48)
- new net RGB_CTRL_2: J2.1 (Pin_1), U2.24 (IO47)
- new net RGB_CTRL_3: J3.1 (Pin_1), U2.26 (IO45)
- new net RGB_CTRL_4: J4.1 (Pin_1), U2.35 (IO42)
- new net RGB_CTRL_5: J5.1 (Pin_1), U2.34 (IO41)
- new net RGB_CTRL_6: J6.1 (Pin_1), U2.33 (IO40)
- new net RGB_CTRL_7: J7.1 (Pin_1), U2.32 (IO39)
- new net RGB_CTRL_8: J8.1 (Pin_1), U2.31 (IO38)
- new net UART_RX: U2.36 (RXD0), U8.6 (TXD)
- new net UART_TX: U2.37 (TXD0), U8.7 (RXD)
- new net USB_D+: U2.14 (USB_D+)
- new net USB_D-: U2.13 (USB_D-)
- no-connect marks 0 -> 1

Commit message: 3
Parts:
- removed J9: Conn_01x03, Connector:FanPinHeader_1x03_P2.54mm_Vertical, symbol Connector_Generic:Conn_01x03
- added C10, C11, C12, C13, C14, C15, C16, C17, C18, C5, C7: 0.1uF, Capacitor_SMD:C_0603_1608Metric_Pad1.08x0.95mm_HandSolder, symbol Device:C_Polarized
- added F4: Fuse, Fuse:Fuse_1206_3216Metric, symbol Device:Fuse
- added J10, J11, J12, J13, J14, J15, J16, J17, J18, J19, J9: Conn_01x02, Connector_JST:JST_SH_BM02B-SRSS-TB_1x02-1MP_P1.00mm_Vertical, symbol Connector_Generic:Conn_01x02
- added J20, J21: Conn_01x04, Connector_PinHeader_2.54mm:PinHeader_1x04_P2.54mm_Vertical, symbol Connector_Generic:Conn_01x04
- added J22: Conn_01x06, Connector_JST:JST_SH_BM06B-SRSS-TB_1x06-1MP_P1.00mm_Vertical, symbol Connector_Generic:Conn_01x06
- added J23: Conn_01x03, Connector_JST:JST_SH_BM03B-SRSS-TB_1x03-1MP_P1.00mm_Vertical, symbol Connector_Generic:Conn_01x03
- added J24: Conn_01x06_Pin, Connector_PinHeader_2.54mm:PinHeader_1x06_P2.54mm_Vertical, symbol Connector:Conn_01x06_Pin
- added R10, R11, R12, R13, R3, R4, R5, R6, R7, R8, R9: 4.7K, Resistor_SMD:R_0805_2012Metric, symbol PCM_Elektuur:R
- added R14, R15, R16, R17: 33Ω, Resistor_SMD:R_0805_2012Metric, symbol PCM_Elektuur:R
- added U1: XT30U-F, XT:CONN-TH_XT30U-M, symbol XT:XT30U-F
- R2: value 1K -> 4.7K; footprint Resistor_SMD:R_1206_3216Metric_Pad1.30x1.75mm_HandSolder -> Resistor_SMD:R_0805_2012Metric
Connections:
- net +3V3: now also R10.1 (+), R11.1 (+), R12.1 (+), R13.1 (+), R3.1 (+), R4.1 (+), R5.1 (+), R6.1 (+), R7.1 (+), R8.1 (+), R9.1 (+)
- net +5V: now also F4.1, J22.1 (Pin_1), J23.1 (Pin_1)
- net D+: now also R16.1 (+)
- net D-: now also R17.1 (+)
- net GND: now also C10.2, C11.2, C12.2, C13.2, C14.2, C15.2, C16.2, C17.2, C18.2, C5.2, C7.2, J10.2 (Pin_2), J11.2 (Pin_2), J12.2 (Pin_2), J13.2 (Pin_2), J14.2 (Pin_2), J15.2 (Pin_2), J16.2 (Pin_2), J17.2 (Pin_2), J18.2 (Pin_2), J19.2 (Pin_2), J20.4 (Pin_4), J21.4 (Pin_4), J22.6 (Pin_6), J23.3 (Pin_3), J9.2 (Pin_2), U1.1 (-)
- net USB_D+: now also R15.1 (+)
- net USB_D-: now also R14.1 (+)
- net UART1_TX: now reaches U2.10 (IO17)
- net UART1_TX: now also J22.2 (Pin_2)
- net UART1_RX: now reaches U2.11 (IO18)
- net UART1_RX: now also J22.3 (Pin_3)
- net BTN_R3: now reaches U2.12 (IO8)
- net BTN_R3: now also C14.1, J15.1 (Pin_1), R9.2 (-)
- net BTN_L2: now reaches U2.15 (IO3)
- net BTN_L2: now also C7.1, J10.1 (Pin_1), R4.2 (-)
- net BTN_Rside: now reaches U2.17 (IO9)
- net BTN_Rside: now also C15.1, J16.1 (Pin_1), R10.2 (-)
- net Key_1: now reaches U2.18 (IO10)
- net Key_1: now also C16.1, J17.1 (Pin_1), R11.2 (-)
- net Key_2: now reaches U2.19 (IO11)
- net Key_2: now also C17.1, J18.1 (Pin_1), R12.2 (-)
- net Key_3: now reaches U2.20 (IO12)
- net Key_3: now also C18.1, J19.1 (Pin_1), R13.2 (-)
- net IO13: now reaches U2.21 (IO13)
- net IO13: now also J24.1 (Pin_1)
- net IO14: now reaches U2.22 (IO14)
- net IO14: now also J24.2 (Pin_2)
- net IO21: now reaches U2.23 (IO21)
- net IO21: now also J24.3 (Pin_3)
- net IO35: now reaches U2.28 (IO35)
- net IO35: now also J24.4 (Pin_4)
- net IO36: now reaches U2.29 (IO36)
- net IO36: now also J24.5 (Pin_5)
- net IO37: now reaches U2.30 (IO37)
- net IO37: now also J24.6 (Pin_6)
- net BTN_L1: now reaches U2.38 (IO2)
- net BTN_L1: now also C5.1, J9.1 (Pin_1), R3.2 (-)
- net BTN_L3: now reaches U2.4 (IO4)
- net BTN_L3: now also C10.1, J11.1 (Pin_1), R5.2 (-)
- net BTN_Lside: now reaches U2.5 (IO5)
- net BTN_Lside: now also C11.1, J12.1 (Pin_1), R6.2 (-)
- net BTN_R1: now reaches U2.6 (IO6)
- net BTN_R1: now also C12.1, J13.1 (Pin_1), R7.2 (-)
- net BTN_R2: now reaches U2.7 (IO7)
- net BTN_R2: now also C13.1, J14.1 (Pin_1), R8.2 (-)
- net Buttun renamed ADC
- net ADC: now also J23.2 (Pin_2)
- new net: J20.3 (Pin_3), R15.2 (-)
- new net: J20.2 (Pin_2), R14.2 (-)
- new net: J21.2 (Pin_2), R16.2 (-)
- new net: J21.3 (Pin_3), R17.2 (-)
- new net +5V_Source: F4.2, J20.1 (Pin_1), J21.1 (Pin_1), U1.2 (+)
- no-connect marks 1 -> 3
Other:
- moved on the sheet: C1, C2, C3, C4, C6, C8, C9, D17, D18, R1, R2, SW1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

Commit message: V1.1
Parts:
- removed C10, C11, C12, C13, C14, C15, C16, C17, C18: 0.1uF, Capacitor_SMD:C_0603_1608Metric_Pad1.08x0.95mm_HandSolder, symbol Device:C_Polarized
- removed J1, J2, J3, J4, J5, J6, J7, J8: Conn_01x03, Connector:FanPinHeader_1x03_P2.54mm_Vertical, symbol Connector_Generic:Conn_01x03
- removed J10, J11, J12, J13, J14, J15, J16, J17, J18, J19, J9: Conn_01x02, Connector_JST:JST_SH_BM02B-SRSS-TB_1x02-1MP_P1.00mm_Vertical, symbol Connector_Generic:Conn_01x02
- removed J23: Conn_01x03, Connector_JST:JST_SH_BM03B-SRSS-TB_1x03-1MP_P1.00mm_Vertical, symbol Connector_Generic:Conn_01x03
- removed J24: Conn_01x06_Pin, Connector_PinHeader_2.54mm:PinHeader_1x06_P2.54mm_Vertical, symbol Connector:Conn_01x06_Pin
- removed R10, R11, R12, R13, R5, R6, R7, R8, R9: 4.7K, Resistor_SMD:R_0805_2012Metric, symbol PCM_Elektuur:R
- removed U1: XT30U-F, XT:CONN-TH_XT30U-M, symbol XT:XT30U-F
- added BTN_L1, BTN_L2, BTN_L3, BTN_R1, BTN_R2, BTN_R3: Conn_01x05, Connector_JST:JST_XH_B5B-XH-AM_1x05_P2.50mm_Vertical, symbol Connector_Generic:Conn_01x05
- added C19, C20, C22, C23, C24, C25, C27, C28: 0.1uF, Capacitor_SMD:C_0603_1608Metric_Pad1.08x0.95mm_HandSolder, symbol Device:C_Polarized
- added Key1, Key2: Conn_01x02, Connector_JST:JST_XH_B2B-XH-AM_1x02_P2.50mm_Vertical, symbol Connector_Generic:Conn_01x02
- added R18, R19, R20, R21, R22, R23, R24, R25: 4.7K, Resistor_SMD:R_0805_2012Metric, symbol PCM_Elektuur:R
Connections:
- net +3V3: now also R18.1 (+), R19.1 (+), R20.1 (+), R21.1 (+), R22.1 (+), R23.1 (+), R24.1 (+), R25.1 (+)
- net +5V: now also BTN_L1.1 (Pin_1), BTN_L2.1 (Pin_1), BTN_L3.1 (Pin_1), BTN_R1.1 (Pin_1), BTN_R2.1 (Pin_1), BTN_R3.1 (Pin_1)
- net BTN_L1: now also BTN_L1.4 (Pin_4), C19.1, R18.2 (-); no longer C5.1, R3.2 (-)
- net BTN_L2: now also BTN_L2.4 (Pin_4), C20.1, R19.2 (-); no longer C7.1, R4.2 (-)
- net BTN_L3: now also BTN_L3.3 (Pin_3), C22.1, R20.2 (-)
- net BTN_Lside: now also BTN_L3.4 (Pin_4), C23.1, R21.2 (-)
- net BTN_R1: now also BTN_R1.4 (Pin_4), C24.1, R22.2 (-)
- net BTN_R2: now also BTN_R2.4 (Pin_4), C25.1, R23.2 (-)
- net BTN_R3: now also BTN_R3.3 (Pin_3), C27.1, R24.2 (-)
- net BTN_Rside: now also BTN_R3.4 (Pin_4), C28.1, R25.2 (-)
- net GND: now also BTN_L1.5 (Pin_5), BTN_L2.5 (Pin_5), BTN_L3.5 (Pin_5), BTN_R1.5 (Pin_5), BTN_R2.5 (Pin_5), BTN_R3.5 (Pin_5), C19.2, C20.2, C22.2, C23.2, C24.2, C25.2, C27.2, C28.2, Key1.2 (Pin_2), Key2.2 (Pin_2)
- net Key_1: now also C5.1, R3.2 (-), Key1.1 (Pin_1)
- net Key_2: now also C7.1, R4.2 (-), Key2.1 (Pin_1)
- net RGB_CTRL_1: now also BTN_L1.2 (Pin_2)
- net RGB_CTRL_5: now also BTN_R1.2 (Pin_2)
- new net: BTN_R1.3 (Pin_3), BTN_R2.2 (Pin_2)
- new net: BTN_L1.3 (Pin_3), BTN_L2.2 (Pin_2)
- new net: BTN_L2.3 (Pin_3), BTN_L3.2 (Pin_2)
- new net: BTN_R2.3 (Pin_3), BTN_R3.2 (Pin_2)
Other:
- moved on the sheet: F4, J20, J21, R14, R15, R16, R17, U8

Commit message: V1.2
Parts:
- removed C6: 0.1uF, Capacitor_SMD:C_0603_1608Metric_Pad1.08x0.95mm_HandSolder, symbol Device:C_Polarized
- removed SW2: SW_DIP_x01, Button_Switch_SMD:SW_SPST_EVQPE1, symbol Switch:SW_DIP_x01
Changed lines of the file:
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@@
 	)
 	(junction
-		(at 113.03 90.17)
-		(diameter 0)
-		(color 0 0 0 0)
-	)
-	(junction
 		(at 133.35 67.31)
 		(diameter 0)
@@
 	(wire
 		(pts
-			(xy 120.65 96.52) (xy 128.27 96.52)
-		)
-		(stroke
-			(width 0)
-			(type default)
-		)
-	)
-	(wire
-		(pts
 			(xy 132.08 102.87) (xy 128.27 102.87)
 		)
@@
 	(wire
 		(pts
-			(xy 128.27 90.17) (xy 128.27 96.52)
-		)
-		(stroke
-			(width 0)
-			(type default)
-		)
-	)
-	(wire
-		(pts
 			(xy 41.91 168.91) (xy 46.99 168.91)
 		)
@@
 	(wire
 		(pts
-			(xy 113.03 90.17) (xy 113.03 96.52)
-		)
-		(stroke
-			(width 0)
-			(type default)
-		)
-	)
-	(wire
-		(pts
 			(xy 242.57 144.78) (xy 242.57 146.05)
 		)
@@
 		)
 	)
-	(label "Boot"
-		(at 128.27 91.44 270)
-		(effects
-			(font
-				(size 1.27 1.27)
-			)
-			(justify right bottom)
-		)
-	)
 	(label "+5V_Source"
 		(at 260.35 132.08 0)
@@
 				)
 				(justify left)
+				(hide yes)
 			)
 		)
@@
 	)
 	(symbol
-		(lib_id "power:GND")
-		(at 113.03 90.17 270)
-		(unit 1)
-		(exclude_from_sim no)
-		(in_bom yes)
-		(on_board yes)
-		(dnp no)
-		(fields_autoplaced yes)
-		(property "Reference" "#PWR09"
-			(at 106.68 90.17 0)
-			(effects
-				(font
-					(size 1.27 1.27)
-				)
-				(hide yes)
-			)
-		)
-		(property "Value" "GND"
-			(at 109.22 90.1699 90)
-			(effects
-				(font
-					(size 1.27 1.27)
-				)
-				(justify right)
-			)
-		)
-		(property "Footprint" ""
-			(at 113.03 90.17 0)
-			(effects
-				(font
-					(size 1.27 1.27)
-				)
-				(hide yes)
-			)
-		)
-		(property "Datasheet" ""
-			(at 113.03 90.17 0)
-			(effects
-				(font
-					(size 1.27 1.27)
-				)
-				(hide yes)
-			)
-		)
-		(property "Description" "Power symbol creates a global label with name \"GND\" , ground"
-			(at 113.03 90.17 0)
-			(effects
-				(font
-					(size 1.27 1.27)
-				)
-				(hide yes)
-			)
-		)
-		(pin "1"
-		)
-		(instances
-			(project "main"
-				(path "/78eeff3e-e2c1-4cc8-997a-22299bf00b85"
-					(reference "#PWR09")
-					(unit 1)
-				)
-			)
-		)
-	)
-	(symbol
 		(lib_id "Device:C_Polarized")
 		(at 87.63 97.79 0)
@@
 	(symbol
 		(lib_id "Device:C_Polarized")
-		(at 116.84 96.52 270)
-		(unit 1)
-		(exclude_from_sim no)
-		(in_bom yes)
-		(on_board yes)
-		(dnp no)
-		(property "Reference" "C6"
-			(at 120.396 93.98 90)
-			(effects
-				(font
-					(size 1.27 1.27)
-				)
-				(justify left)
-			)
-		)
-		(property "Value" "0.1uF"
-			(at 120.396 95.504 90)
-			(effects
-				(font
-					(size 1.27 1.27)
-				)
-				(justify left)
-			)
-		)
-		(property "Footprint" "Capacitor_SMD:C_0603_1608Metric_Pad1.08x0.95mm_HandSolder"
-			(at 113.03 97.4852 0)
-			(effects
-				(font
-					(size 1.27 1.27)
-				)
-				(hide yes)
-			)
-		)
-		(property "Datasheet" "~"
-			(at 116.84 96.52 0)
-			(effects
-				(font
-					(size 1.27 1.27)
-				)
-				(hide yes)
-			)
-		)
-		(property "Description" "Polarized capacitor"
-			(at 116.84 96.52 0)
-			(effects
-				(font
-					(size 1.27 1.27)
-				)
-				(hide yes)
-			)
-		)
-		(pin "1"
-		)
-		(pin "2"
-		)
-		(instances
-			(project "main"
-				(path "/78eeff3e-e2c1-4cc8-997a-22299bf00b85"
-					(reference "C6")
-					(unit 1)
-				)
-			)
-		)
-	)
-	(symbol
-		(lib_id "Device:C_Polarized")
 		(at 26.67 31.75 0)
 		(unit 1)
@@
 					(unit 1)
 				)
-			)
-		)
-	)
-	(symbol
-		(lib_id "Switch:SW_DIP_x01")
-		(at 120.65 90.17 0)
-		(unit 1)
-		(exclude_from_sim no)
-		(in_bom yes)
-		(on_board yes)
-		(dnp no)
-		(property "Reference" "SW2"
-			(at 120.904 86.36 0)
-			(effects
-				(font
-					(size 1.27 1.27)
-				)
-			)
-		)
-		(property "Value" "SW_DIP_x01"
-			(at 120.65 85.09 0)
-			(effects
-				(font
-					(size 1.27 1.27)
-				)
-				(hide yes)
-			)
-		)
-		(property "Footprint" "Button_Switch_SMD:SW_SPST_EVQPE1"
-			(at 120.65 90.17 0)
-			(effects
-				(font
-					(size 1.27 1.27)
-				)
-				(hide yes)
-			)
-		)
-		(property "Datasheet" "~"
-			(at 120.65 90.17 0)
-			(effects
-				(font
-					(size 1.27 1.27)
-				)
-				(hide yes)
-			)
-		)
-		(property "Description" "1x DIP Switch, Single Pole Single Throw (SPST) switch, small symbol"
-			(at 120.65 90.17 0)
-			(effects
-				(font
-					(size 1.27 1.27)
-				)
-				(hide yes)
-			)
-		)
-		(pin "2"
-		)
-		(pin "1"
-		)
-		(instances
-			(project "main"
-				(path "/78eeff3e-e2c1-4cc8-997a-22299bf00b85"
-					(reference "SW2")
-					(unit 1)
-				)

Commit message: V1.21
Parts:
- added SW2: SW_DIP_x01, Button_Switch_SMD:SW_SPST_EVQPE1, symbol Switch:SW_DIP_x01
- J20: footprint Connector_PinHeader_2.54mm:PinHeader_1x04_P2.54mm_Vertical -> Connector_JST:JST_XH_B4B-XH-A_1x04_P2.50mm_Vertical
Connections:
- net +5V_Source: now also J20.4 (Pin_4); no longer J20.1 (Pin_1)
- net Boot: now also SW2.2
- net GND: now also J20.1 (Pin_1), SW2.1; no longer J20.4 (Pin_4)
Other:
- moved on the sheet: F4
Changed lines of the file:
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@@
 	(wire
 		(pts
-			(xy 266.7 107.95) (xy 273.05 107.95)
+			(xy 266.7 127) (xy 273.05 127)
 		)
 		(stroke
@@
 	(wire
 		(pts
+			(xy 273.05 120.65) (xy 273.05 127)
+		)
+		(stroke
+			(width 0)
+			(type default)
+		)
+	)
+	(wire
+		(pts
 			(xy 271.78 132.08) (xy 271.78 135.89)
 		)
@@
 	(wire
 		(pts
+			(xy 127 90.17) (xy 132.08 90.17)
+		)
+		(stroke
+			(width 0)
+			(type default)
+		)
+	)
+	(wire
+		(pts
 			(xy 26.67 27.94) (xy 27.94 27.94)
 		)
@@
 	(wire
 		(pts
-			(xy 273.05 107.95) (xy 273.05 113.03)
-		)
-		(stroke
-			(width 0)
-			(type default)
-		)
-	)
-	(wire
-		(pts
 			(xy 50.8 161.29) (xy 46.99 161.29)
 		)
@@
 	)
 	(label "+5V_Source"
-		(at 266.7 107.95 0)
+		(at 266.7 127 0)
 		(effects
 			(font
@@
 		)
 	)
+	(label "Boot"
+		(at 132.08 90.17 180)
+		(effects
+			(font
+				(size 1.27 1.27)
+			)
+			(justify right bottom)
+		)
+	)
 	(label "BTN_L2"
 		(at 29.21 69.85 0)
@@
 	)
 	(symbol
+		(lib_id "Switch:SW_DIP_x01")
+		(at 119.38 90.17 0)
+		(unit 1)
+		(exclude_from_sim no)
+		(in_bom yes)
+		(on_board yes)
+		(dnp no)
+		(property "Reference" "SW2"
+			(at 115.57 86.36 0)
+			(effects
+				(font
+					(size 1.27 1.27)
+				)
+			)
+		)
+		(property "Value" "SW_DIP_x01"
+			(at 119.38 85.09 0)
+			(effects
+				(font
+					(size 1.27 1.27)
+				)
+				(hide yes)
+			)
+		)
+		(property "Footprint" "Button_Switch_SMD:SW_SPST_EVQPE1"
+			(at 119.38 90.17 0)
+			(effects
+				(font
+					(size 1.27 1.27)
+				)
+				(hide yes)
+			)
+		)
+		(property "Datasheet" "~"
+			(at 119.38 90.17 0)
+			(effects
+				(font
+					(size 1.27 1.27)
+				)
+				(hide yes)
+			)
+		)
+		(property "Description" "1x DIP Switch, Single Pole Single Throw (SPST) switch, small symbol"
+			(at 119.38 90.17 0)
+			(effects
+				(font
+					(size 1.27 1.27)
+				)
+				(hide yes)
+			)
+		)
+		(pin "2"
+		)
+		(pin "1"
+		)
+		(instances
+			(project "main"
+				(path "/78eeff3e-e2c1-4cc8-997a-22299bf00b85"
+					(reference "SW2")
+					(unit 1)
+				)
+			)
+		)
+	)
+	(symbol
 		(lib_id "power:+3V3")
 		(at 228.6 68.58 0)
@@
 	(symbol
 		(lib_id "power:GND")
-		(at 273.05 120.65 0)
+		(at 273.05 113.03 180)
 		(unit 1)
 		(exclude_from_sim no)
@@
 		(fields_autoplaced yes)
 		(property "Reference" "#PWR082"
-			(at 273.05 127 0)
+			(at 273.05 106.68 0)
 			(effects
 				(font
@@
 		)
 		(property "Value" "GND"
-			(at 273.05 125.73 0)
+			(at 273.05 107.95 0)
 			(effects
 				(font
@@
 		)
 		(property "Footprint" ""
-			(at 273.05 120.65 0)
+			(at 273.05 113.03 0)
 			(effects
 				(font
@@
 		)
 		(property "Datasheet" ""
-			(at 273.05 120.65 0)
+			(at 273.05 113.03 0)
 			(effects
 				(font
@@
 		)
 		(property "Description" "Power symbol creates a global label with name \"GND\" , ground"
-			(at 273.05 120.65 0)
+			(at 273.05 113.03 0)
 			(effects
 				(font
@@
 	(symbol
 		(lib_id "Device:Fuse")
-		(at 262.89 107.95 90)
+		(at 262.89 127 90)
 		(unit 1)
 		(exclude_from_sim no)
@@
 		(dnp no)
 		(property "Reference" "F4"
-			(at 262.89 104.394 90)
+			(at 262.89 129.032 90)
 			(effects
 				(font
@@
 		)
 		(property "Value" "Fuse"
-			(at 262.89 106.172 90)
+			(at 262.89 125.222 90)
 			(effects
 				(font
@@
 		)
 		(property "Footprint" "Fuse:Fuse_1206_3216Metric"
-			(at 262.89 109.728 90)
+			(at 262.89 128.778 90)
 			(effects
 				(font
@@
 		)
 		(property "Datasheet" "~"
-			(at 262.89 107.95 0)
+			(at 262.89 127 0)
 			(effects
 				(font
@@
 		)
 		(property "Description" "Fuse"
-			(at 262.89 107.95 0)
+			(at 262.89 127 0)
 			(effects
 				(font
@@
 	)
 	(symbol
+		(lib_id "power:GND")
+		(at 111.76 90.17 270)
+		(unit 1)
+		(exclude_from_sim no)
+		(in_bom yes)
+		(on_board yes)
+		(dnp no)
+		(fields_autoplaced yes)
+		(property "Reference" "#PWR09"
+			(at 105.41 90.17 0)
+			(effects
+				(font
+					(size 1.27 1.27)
+				)
+				(hide yes)
+			)
+		)
+		(property "Value" "GND"
+			(at 107.95 90.1699 90)
+			(effects
+				(font
+					(size 1.27 1.27)
+				)
+				(justify right)
+			)
+		)
+		(property "Footprint" ""
+			(at 111.76 90.17 0)
+			(effects
+				(font
+					(size 1.27 1.27)
+				)
+				(hide yes)
+			)
+		)
+		(property "Datasheet" ""
+			(at 111.76 90.17 0)
+			(effects
+				(font
+					(size 1.27 1.27)
+				)
+				(hide yes)
+			)
+		)
+		(property "Description" "Power symbol creates a global label with name \"GND\" , ground"
+			(at 111.76 90.17 0)
+			(effects
+				(font
+					(size 1.27 1.27)
+				)
+				(hide yes)
+			)
+		)
+		(pin "1"
+		)
+		(instances
+			(project "main"
+				(path "/78eeff3e-e2c1-4cc8-997a-22299bf00b85"
+					(reference "#PWR09")
+					(unit 1)
+				)
+			)
+		)
+	)
+	(symbol
 		(lib_id "Device:C_Polarized")
 		(at 40.64 95.25 0)
@@
 			)
 		)
-		(property "Footprint" "Connector_PinHeader_2.54mm:PinHeader_1x04_P2.54mm_Vertical"
+		(property "Footprint" "Connector_JST:JST_XH_B4B-XH-A_1x04_P2.50mm_Vertical"
 			(at 278.13 115.57 0)
 			(effects
@@
 	(symbol
 		(lib_id "power:+5V")
-		(at 259.08 107.95 90)
+		(at 259.08 127 90)
 		(unit 1)
 		(exclude_from_sim no)
@@
 		(fields_autoplaced yes)
 		(property "Reference" "#PWR081"
-			(at 262.89 107.95 0)
+			(at 262.89 127 0)
 			(effects
 				(font
@@
 		)
 		(property "Value" "+5V"
-			(at 255.27 107.9499 90)
+			(at 255.27 126.9999 90)
 			(effects
 				(font
@@
 		)
 		(property "Footprint" ""
-			(at 259.08 107.95 0)
+			(at 259.08 127 0)
 			(effects
 				(font
@@
 		)
 		(property "Datasheet" ""
-			(at 259.08 107.95 0)
+			(at 259.08 127 0)
 			(effects
 				(font
@@
 		)
 		(property "Description" "Power symbol creates a global label with name \"+5V\""
-			(at 259.08 107.95 0)
+			(at 259.08 127 0)
 			(effects
 				(font
